File: Circuit_layout.kicad_pcb (KiCad board)
At the start: 2 copper layers, 154.9 x 131.6 mm, 82 parts, among them J1 ICSP, J10 Conn_BoardJ6, J11 RTDS, J12 Conn_BoardJ7, J13 Conn_BoardJ8, J14 Conn_BoardJ21, J15 Conn_BoardJ24, J2 Chip_conn1, J23 Testing_pins, J24 24v_Banana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

Commit message: addition conn for external pedal
Parts:
- removed G***: LOGO, custom_footprints:logo_lafayette_ece_24mmx9mm
- removed REF** (x4): MountingHole_3.5mm_Pad, custom_footprints:MountingHole_3.5mm_Pad
- removed VAL: REF, custom_footprints:lafLogo
- added J16: APPS2_External, Connectors_Molex:Molex_MiniFit-JR-5556-02A_2x01x4.20mm_Straight, F.Cu at (114.0, 133.3)
- added J17: APPS1_External, Connectors_Molex:Molex_MiniFit-JR-5556-02A_2x01x4.20mm_Straight, F.Cu at (36.3, 133.3)
- added JP7: Jumper_NC_Dual, Pin_Headers:Pin_Header_Straight_1x03_Pitch2.54mm, F.Cu at (104.6, 138.7)
- added JP8: Jumper_NC_Dual, Pin_Headers:Pin_Header_Straight_1x03_Pitch2.54mm, F.Cu at (46.5, 134.4)
- D8: value Safty_Loop_LED -> Safety_Loop_LED
- moved JP3 9.14 mm to (93.5, 126.5)
- moved JP5 6.60 mm to (65.0, 126.5)
- moved JP4 5.59 mm to (104.1, 126.5)
- moved D9 5.32 mm to (110.5, 118.4)
- moved JP6 5.08 mm to (52.8, 126.5)
- moved R11 4.91 mm to (110.5, 113.3), turned to 180 degrees
- moved R13 4.62 mm to (104.9, 98.6)
- moved D13 4.41 mm to (95.9, 119.1), turned to 180 degrees
- moved D11 4.38 mm to (104.9, 102.9), turned to 180 degrees
- moved R9 4.33 mm to (88.6, 98.0), turned to 0 degrees
- moved R15 4.22 mm to (96.0, 114.8)
- moved D7 4.08 mm to (88.6, 102.1)
- moved R14 4.07 mm to (82.3, 114.0), turned to 0 degrees
- moved R12 3.93 mm to (68.1, 114.0)
- moved D10 3.86 mm to (68.1, 117.9), turned to 180 degrees
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Connections:
- net /Drive_BTN_5v renamed /Drive_BTN_RTN
- D10 pad 1: /BP -> /BP_RTN
- D11 pad 1: /SPARE_LED -> /SPARE_LED_RTN
- D12 pad 1: /IMD_Fault_LED -> /IMD_Fault_RTN
- D13 pad 1: /TSAL_Cock -> /TSAL_Cock_RTN
- D7 pad 1: /TSAL_1 -> /TSAL_1_RTN
- D8 pad 1: Net-(D8-Pad1) -> /SL1
- D9 pad 1: /Drive_LED -> /Drive_LED_RTN
- JP3 pad 2: /APPS2 -> Net-(JP3-Pad2)
- JP5 pad 2: /APPS1 -> Net-(JP5-Pad2)
- R10 pad 1: /SL1 -> Net-(D8-Pad2)
- R10 pad 2: Net-(D8-Pad2) -> Net-(R10-Pad2)
- R11 pad 1: /Drive_LED_RTN -> Net-(D9-Pad2)
- R11 pad 2: Net-(D9-Pad2) -> /Drive_LED
- R12 pad 1: /BP_RTN -> Net-(D10-Pad2)
- R12 pad 2: Net-(D10-Pad2) -> /BP
- R13 pad 1: /SPARE_LED_RTN -> Net-(D11-Pad2)
- R13 pad 2: Net-(D11-Pad2) -> /SPARE_LED
- R14 pad 1: /IMD_Fault_RTN -> Net-(D12-Pad2)
- R14 pad 2: Net-(D12-Pad2) -> /IMD_Fault_LED
- R15 pad 1: /TSAL_Cock_RTN -> Net-(D13-Pad2)
- R15 pad 2: Net-(D13-Pad2) -> /TSAL_Cock
- R9 pad 1: /TSAL_1_RTN -> Net-(D7-Pad2)
- R9 pad 2: Net-(D7-Pad2) -> /TSAL_1
- SW2 pad 3: Net-(D8-Pad1) -> Net-(R10-Pad2)
Routing:
- net /APPS2_5: track 93.4 -> 136.2 mm, vias 3 -> 5
- net Net-(R10-Pad2): track 0.00 -> 34.6 mm
- net Net-(D8-Pad1): track 34.6 -> 0.00 mm
- net /APPS1: track 153.7 -> 179.7 mm, vias 6 -> 8
- net Net-(JP5-Pad2): track 0.00 -> 23.9 mm, vias 0 -> 1
- net Net-(JP3-Pad2): track 0.00 -> 20.8 mm, vias 0 -> 1
- net Net-(J17-Pad1): track 0.00 -> 16.6 mm
- net /APPS2: track 240.7 -> 254.7 mm
- net Net-(J16-Pad1): track 0.00 -> 12.6 mm
- net /APPS1_10: track 146.5 -> 158.0 mm, vias 1 -> 6
- net /APPS2_RTN: track 162.1 -> 150.9 mm
- net Net-(JP4-Pad3): track 24.4 -> 34.9 mm, vias 0 -> 2
- net Net-(JP3-Pad1): track 19.0 -> 10.5 mm
- net Net-(JP6-Pad1): track 44.2 -> 39.2 mm
- net Net-(JP5-Pad1): track 27.7 -> 23.2 mm
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Other:
- net class Default: clearance 0.254 -> 0.2
- rule trace_clearance: 0.254 -> 0.2
- board text added: "EXT"
- board text added: "INT"
- board text added: "J1"
- board text added: "SAFETY LOOP"
